Commit message: quaternion

File: src/kinematics/urdf/simple_robot.urdf (robot description, URDF)
Before this commit: robot simple_robot, 7 links, 6 joints
Joints:
- joint joint2: axis 0 1 0 -> 0 -1 0
- joint joint3: axis 0 1 0 -> 0 -1 0
- joint joint4: type revolute -> fixed
- joint joint5: type revolute -> fixed
- joint joint6: type revolute -> fixed

Commit message: 5 dof

File: src/kinematics/urdf/simple_robot.urdf (robot description, URDF)
Before this commit: robot simple_robot, 7 links, 6 joints
Links:
- link link3: geometry visual cylinder length=0.06 radius=0.04
- link link5: geometry visual cylinder length=0.06 radius=0.04
- link link6: geometry visual box size=0.04 0.04 0.01
Joints:
- joint joint1: axis 0 0 -1 -> 0 0 1
- joint joint2: origin xyz=0 0 0.4 -> xyz=0 0.05 0.4
- joint joint4: origin xyz=0.1 0 0 -> xyz=0.06 0 0; type fixed -> revolute
- joint joint5: axis 0 1 0 -> 0 -1 0; type fixed -> revolute
- joint joint6: origin xyz=0.1 0 0 -> xyz=0.06 0 0
